Commit message: fix

File: cylinder.urdf (robot description, URDF)
Before this commit: robot cylinder, 2 links, 1 joints
Joints:
- joint joint_base_head: origin xyz=-0.1414 -0.1414 0 -> xyz=0 0.2 0.1

File: cylinder2.urdf (robot description, URDF)
Before this commit: robot cylinder, 2 links, 1 joints
Joints:
- joint joint_base_head: origin xyz=-0.1414 -0.1414 0 -> xyz=0 0.2 0.1
